Commit message: Updated deepfind distance, launch files and deepfind URDF

File: catkin_ws/src/deepfind_navigation/urdf/deepfind.urdf (robot description, URDF)
Before this commit: robot deepfind, 8 links, 7 joints
Links:
- removed link lower_base
- added link base_link, mass 0.00205673; collision box size=0.27676 0.34582 0.021538; visual box size=0.27676 0.34582 0.021538
- link ball_caster_box: mass 0.000286893 -> 0.000704419; geometry collision box size=0.127232 0.083214 0.066526; visual box size=0.127232 0.083214 0.066526
- link left_wall: mass 0.000704419 -> 0.000286893; geometry collision box size=0.018328 0.212902 0.073543; visual box size=0.018328 0.212902 0.073543
Joints:
- removed joint ball_caster_to_box
- removed joint left_right_wheels
- removed joint left_wall_bc
- removed joint left_wheel_left_wall
- removed joint left_wheel_lower_base
- removed joint left_wheel_right_wall
- removed joint left_wheel_upper_base
- added joint base_link_bc: type fixed, parent base_link, child ball_caster, origin xyz=0 0 0
- added joint base_link_bc_box: type fixed, parent base_link, child ball_caster_box, origin xyz=0 0 0
- added joint base_link_left: type fixed, parent base_link, child left_wheel, origin xyz=0 0 0
- added joint base_link_left_wall: type fixed, parent base_link, child left_wall, origin xyz=0 0 0
- added joint base_link_right: type fixed, parent base_link, child right_wheel, origin xyz=0 0 0
- added joint base_link_right_wall: type fixed, parent base_link, child right_wall, origin xyz=0 0 0
- added joint base_link_upper: type fixed, parent base_link, child upper_base, origin xyz=0 0 0
